Commit message: Still debugging the IK

File: src/mildred_description/urdf/macros.xacro (robot description, xacro)
@@ -1,8 +1,69 @@
 <robot xmlns:xacro="http://www.ros.org/wiki/xacro">
+    <!--<xacro:macro name="default_inertial" params="mass">-->
+        <!--<inertial>-->
+            <!--<mass value="${mass}"/>-->
+            <!--&lt;!&ndash;<inertia ixx="1.0" ixy="0.0" ixz="0.0" iyy="1.0" iyz="0.0" izz="1.0" />&ndash;&gt;-->
+            <!--<inertia ixx="0.001" ixy="0.0" ixz="0.0" iyy="0.001" iyz="0.0" izz="0.001"/>-->
+        <!--</inertial>-->
+    <!--</xacro:macro>-->
+    <!--<xacro:macro name="sphere_inertial" params="radius mass">-->
+        <!--<inertial>-->
+            <!--<mass value="${mass}" />-->
+            <!--<origin xyz="0 0 0" />-->
+            <!--<inertia ixx="${0.4 * mass * radius * radius}" ixy="0.0" ixz="0.0"-->
+                     <!--iyy="${0.4 * mass * radius * radius}" iyz="0.0"-->
+                     <!--izz="${0.4 * mass * radius * radius}" />-->
+        <!--</inertial>-->
+    <!--</xacro:macro>-->
+    <!--<xacro:macro name="cylinder_inertial" params="radius length mass">-->
+        <!--<inertial>-->
+            <!--<mass value="${mass}" />-->
+            <!--<origin xyz="0 0 0" />-->
+            <!--<inertia ixx="${0.0833333 * mass * (3 * radius * radius + length * length)}" ixy="0.0" ixz="0.0"-->
+                     <!--iyy="${0.0833333 * mass * (3 * radius * radius + length * length)}" iyz="0.0"-->
+                     <!--izz="${0.5 * mass * radius * radius}" />-->
+        <!--</inertial>-->
+    <!--</xacro:macro>-->
+    <!--<xacro:macro name="box_inertial" params="x y z mass">-->
+        <!--<inertial>-->
+            <!--<mass value="${mass}" />-->
+            <!--<origin xyz="0 0 0" />-->
+            <!--<inertia ixx="${0.0833333 * mass * (y*y + z*z)}" ixy="0.0" ixz="0.0"-->
+                     <!--iyy="${0.0833333 * mass * (x*x + z*z)}" iyz="0.0"-->
+                     <!--izz="${0.0833333 * mass * (x*x + y*y)}" />-->
+        <!--</inertial>-->
+    <!--</xacro:macro>-->
+    <!--<xacro:macro name="sphere_inertial_with_origin" params="radius mass *origin">-->
+        <!--<inertial>-->
+            <!--<mass value="${mass}" />-->
+            <!--<xacro:insert_block name="origin" />-->
+            <!--<inertia ixx="${0.4 * mass * radius * radius}" ixy="0.0" ixz="0.0"-->
+                     <!--iyy="${0.4 * mass * radius * radius}" iyz="0.0"-->
+                     <!--izz="${0.4 * mass * radius * radius}" />-->
+        <!--</inertial>-->
+    <!--</xacro:macro>-->
+    <!--<xacro:macro name="cylinder_inertial_with_origin" params="radius length mass *origin">-->
+        <!--<inertial>-->
+            <!--<mass value="${mass}" />-->
+            <!--<xacro:insert_block name="origin" />-->
+            <!--<inertia ixx="${0.0833333 * mass * (3 * radius * radius + length * length)}" ixy="0.0" ixz="0.0"-->
+                     <!--iyy="${0.0833333 * mass * (3 * radius * radius + length * length)}" iyz="0.0"-->
+                     <!--izz="${0.5 * mass * radius * radius}" />-->
+        <!--</inertial>-->
+    <!--</xacro:macro>-->
+    <!--<xacro:macro name="box_inertial_with_origin" params="x y z mass *origin">-->
+        <!--<inertial>-->
+            <!--<mass value="${mass}" />-->
+            <!--<xacro:insert_block name="origin" />-->
+            <!--<inertia ixx="${0.0833333 * mass * (y*y + z*z)}" ixy="0.0" ixz="0.0"-->
+                     <!--iyy="${0.0833333 * mass * (x*x + z*z)}" iyz="0.0"-->
+                     <!--izz="${0.0833333 * mass * (x*x + y*y)}" />-->
+        <!--</inertial>-->
+    <!--</xacro:macro>-->
     <xacro:macro name="default_inertial" params="mass">
         <inertial>
             <mass value="${mass}"/>
             <!--<inertia ixx="1.0" ixy="0.0" ixz="0.0" iyy="1.0" iyz="0.0" izz="1.0" />-->
-            <inertia ixx="0.001" ixy="0.0" ixz="0.0" iyy="0.001" iyz="0.0" izz="0.001"/>
+            <inertia ixx="1.0" ixy="0.0" ixz="0.0" iyy="1.0" iyz="0.0" izz="1.0"/>
         </inertial>
     </xacro:macro>
@@ -11,7 +72,7 @@
             <mass value="${mass}" />
             <origin xyz="0 0 0" />
-            <inertia ixx="${0.4 * mass * radius * radius}" ixy="0.0" ixz="0.0"
-                     iyy="${0.4 * mass * radius * radius}" iyz="0.0"
-                     izz="${0.4 * mass * radius * radius}" />
+            <inertia ixx="1.0" ixy="0.0" ixz="0.0"
+                     iyy="1.0" iyz="0.0"
+                     izz="1.0" />
         </inertial>
     </xacro:macro>
@@ -20,7 +81,7 @@
             <mass value="${mass}" />
             <origin xyz="0 0 0" />
-            <inertia ixx="${0.0833333 * mass * (3 * radius * radius + length * length)}" ixy="0.0" ixz="0.0"
-                     iyy="${0.0833333 * mass * (3 * radius * radius + length * length)}" iyz="0.0"
-                     izz="${0.5 * mass * radius * radius}" />
+            <inertia ixx="1.0" ixy="0.0" ixz="0.0"
+                     iyy="1.0" iyz="0.0"
+                     izz="1.0" />
         </inertial>
     </xacro:macro>
@@ -29,7 +90,7 @@
             <mass value="${mass}" />
             <origin xyz="0 0 0" />
-            <inertia ixx="${0.0833333 * mass * (y*y + z*z)}" ixy="0.0" ixz="0.0"
-                     iyy="${0.0833333 * mass * (x*x + z*z)}" iyz="0.0"
-                     izz="${0.0833333 * mass * (x*x + y*y)}" />
+            <inertia ixx="1.0" ixy="0.0" ixz="0.0"
+                     iyy="1.0" iyz="0.0"
+                     izz="1.0" />
         </inertial>
     </xacro:macro>
@@ -38,7 +99,7 @@
             <mass value="${mass}" />
             <xacro:insert_block name="origin" />
-            <inertia ixx="${0.4 * mass * radius * radius}" ixy="0.0" ixz="0.0"
-                     iyy="${0.4 * mass * radius * radius}" iyz="0.0"
-                     izz="${0.4 * mass * radius * radius}" />
+            <inertia ixx="1.0" ixy="0.0" ixz="0.0"
+                     iyy="1.0" iyz="0.0"
+                     izz="1.0" />
         </inertial>
     </xacro:macro>
@@ -47,7 +108,7 @@
             <mass value="${mass}" />
             <xacro:insert_block name="origin" />
-            <inertia ixx="${0.0833333 * mass * (3 * radius * radius + length * length)}" ixy="0.0" ixz="0.0"
-                     iyy="${0.0833333 * mass * (3 * radius * radius + length * length)}" iyz="0.0"
-                     izz="${0.5 * mass * radius * radius}" />
+            <inertia ixx="1.0" ixy="0.0" ixz="0.0"
+                     iyy="1.0" iyz="0.0"
+                     izz="1.0" />
         </inertial>
     </xacro:macro>
@@ -56,7 +117,7 @@
             <mass value="${mass}" />
             <xacro:insert_block name="origin" />
-            <inertia ixx="${0.0833333 * mass * (y*y + z*z)}" ixy="0.0" ixz="0.0"
-                     iyy="${0.0833333 * mass * (x*x + z*z)}" iyz="0.0"
-                     izz="${0.0833333 * mass * (x*x + y*y)}" />
+            <inertia ixx="1.0" ixy="0.0" ixz="0.0"
+                     iyy="1.0" iyz="0.0"
+                     izz="1.0" />
         </inertial>
     </xacro:macro>

File: src/mildred_description/urdf/variables.xacro (robot description, xacro)
@@ -6,12 +6,12 @@
     <xacro:property name="thorax_radius" value="0.064"/>
     <xacro:property name="thorax_height" value="0.040"/>
+    <xacro:property name="thorax_mass" value="0.2"/>
     <xacro:property name="coxa_length" value="0.03525"/>
+    <xacro:property name="coxa_mass" value="0.162"/>
     <xacro:property name="femur_length" value="0.0975"/>
     <xacro:property name="femur_angle" value="39.2"/>
+    <xacro:property name="femur_mass" value="0.025981"/>
     <xacro:property name="tibia_length" value="0.195"/>
     <xacro:property name="tibia_angle" value="21.3"/>
-    <xacro:property name="thorax_mass" value="0.2"/>
-    <xacro:property name="coxa_mass" value="0.162"/>
-    <xacro:property name="femur_mass" value="0.025981"/>
     <xacro:property name="tibia_mass" value="0.107208"/>
     <xacro:property name="foot_radius" value="0.012"/>
@@ -23,5 +23,5 @@
     <!--<xacro:property name="foot_mass" value="1.0"/>-->
     <!-- http://emanual.robotis.com/docs/en/dxl/x/xl430-w250/#specifications -->
-    <xacro:property name="max_torque" value="1.4"/> <!-- this is stall torque, graph shows 0.84 -->
+    <xacro:property name="max_torque" value="100.4"/> <!-- this is stall torque, graph shows 0.84 -->
     <xacro:property name="max_velocity" value="${((2*pi)/60)*57}"/> <!-- rpm to rad/s -->
     <!--<xacro:property name="max_torque" value="10000"/> &lt;!&ndash; fuck it, just move &ndash;&gt;-->

Commit message: I guess this can be called progress

File: src/mildred_description/urdf/macros.xacro (robot description, xacro)
@@ -1,3 +1,16 @@
 <robot xmlns:xacro="http://www.ros.org/wiki/xacro">
+    <xacro:macro name="default_inertial">
+        <inertial>
+            <origin xyz="0.0 0.0 0.0" rpy="0.0 0.0 0.0" />
+            <mass value="0.00001"/>
+            <inertia ixx="1.0" ixy="0.0" ixz="0.0" iyy="1.0" iyz="0.0" izz="1.0"/>
+        </inertial>
+    </xacro:macro>
+    <xacro:macro name="default_inertial_mass" params="mass">
+        <inertial>
+            <mass value="${mass}"/>
+            <inertia ixx="1.0" ixy="0.0" ixz="0.0" iyy="1.0" iyz="0.0" izz="1.0"/>
+        </inertial>
+    </xacro:macro>
     <!--<xacro:macro name="default_inertial" params="mass">-->
         <!--<inertial>-->
@@ -61,11 +74,4 @@
         <!--</inertial>-->
     <!--</xacro:macro>-->
-    <xacro:macro name="default_inertial" params="mass">
-        <inertial>
-            <mass value="${mass}"/>
-            <!--<inertia ixx="1.0" ixy="0.0" ixz="0.0" iyy="1.0" iyz="0.0" izz="1.0" />-->
-            <inertia ixx="1.0" ixy="0.0" ixz="0.0" iyy="1.0" iyz="0.0" izz="1.0"/>
-        </inertial>
-    </xacro:macro>
     <xacro:macro name="sphere_inertial" params="radius mass">
         <inertial>

File: src/mildred_description/urdf/mildred.urdf.xacro (robot description, xacro)
@@ -29,5 +29,6 @@
             </geometry>
         </collision>
-        <xacro:default_inertial mass="${thorax_mass}"/>
+        <xacro:default_inertial/>
+        <!--<xacro:default_inertial mass="${thorax_mass}"/>-->
     </link>
     <gazebo reference="thorax">
@@ -43,5 +44,5 @@
             <axis xyz="0.00 0.00 1.00"/>
             <limit lower="${TC_joint_lower_limit}" upper="${TC_joint_upper_limit}" effort="${max_torque}" velocity="${max_velocity}"/>
-            <dynamics damping="${damping}" friction="${friction}" />
+            <!--<dynamics damping="${damping}" friction="${friction}" />-->
         </joint>
         <link name="coxa_${suffix}">
@@ -61,19 +62,30 @@
                 </geometry>
             </collision>
-            <xacro:cylinder_inertial_with_origin mass="${coxa_mass}" radius="0.02" length="${coxa_length}">
-                <origin xyz="${coxa_length/2} 0.00 0.00" rpy="0.00 ${radians(90)} 0.00"/>
-            </xacro:cylinder_inertial_with_origin>
+            <xacro:default_inertial/>
+            <!--<xacro:cylinder_inertial_with_origin mass="${coxa_mass}" radius="0.02" length="${coxa_length}">-->
+                <!--<origin xyz="${coxa_length/2} 0.00 0.00" rpy="0.00 ${radians(90)} 0.00"/>-->
+            <!--</xacro:cylinder_inertial_with_origin>-->
         </link>
         <gazebo reference="coxa_${suffix}">
             <material>Gazebo/Blue</material>
         </gazebo>
+        <transmission name="TC_trans_${suffix}">
+            <type>transmission_interface/SimpleTransmission</type>
+            <joint name="TC_joint_${suffix}">
+                <hardwareInterface>hardware_interface/EffortJointInterface</hardwareInterface>
+            </joint>
+            <actuator name="TC_motor_${suffix}">
+                <hardwareInterface>hardware_interface/EffortJointInterface</hardwareInterface>
+                <mechanicalReduction>1</mechanicalReduction>
+            </actuator>
+        </transmission>
         <!-- Link 2/Femur -->
         <joint name="CF_joint_${suffix}" type="revolute">
             <parent link="coxa_${suffix}"/>
             <child link="femur_${suffix}"/>
-            <origin xyz="${coxa_length} 0.00 0.00" rpy="0.00 ${-radians(femur_angle)} 0.00"/>
-            <axis xyz="0.00 ${mirror * -1.00} 0.00"/>
+            <origin xyz="${coxa_length} 0.00 0.00" rpy="0.00 0.00 0.00"/>
+            <axis xyz="0.00 1.00 0.00"/>
             <limit lower="${CF_joint_lower_limit}" upper="${CF_joint_upper_limit}" effort="${max_torque}" velocity="${max_velocity}"/>
-            <dynamics damping="${damping}" friction="${friction}" />
+            <!--<dynamics damping="${damping}" friction="${friction}" />-->
         </joint>
         <link name="femur_${suffix}">
@@ -93,19 +105,30 @@
                 </geometry>
             </collision>
-            <xacro:cylinder_inertial_with_origin mass="${femur_mass}" radius="0.02" length="${femur_length}">
-                <origin xyz="${femur_length/2} 0.00 0.00" rpy="0.00 ${radians(90)} 0.00"/>
-            </xacro:cylinder_inertial_with_origin>
+            <xacro:default_inertial/>
+            <!--<xacro:cylinder_inertial_with_origin mass="${femur_mass}" radius="0.02" length="${femur_length}">-->
+                <!--<origin xyz="${femur_length/2} 0.00 0.00" rpy="0.00 ${radians(90)} 0.00"/>-->
+            <!--</xacro:cylinder_inertial_with_origin>-->
         </link>
         <gazebo reference="femur_${suffix}">
             <material>Gazebo/Turquoise</material>
         </gazebo>
+        <transmission name="CF_trans_${suffix}">
+            <type>transmission_interface/SimpleTransmission</type>
+            <joint name="CF_joint_${suffix}">
+                <hardwareInterface>hardware_interface/EffortJointInterface</hardwareInterface>
+            </joint>
+            <actuator name="CF_motor_${suffix}">
+                <hardwareInterface>hardware_interface/EffortJointInterface</hardwareInterface>
+                <mechanicalReduction>1</mechanicalReduction>
+            </actuator>
+        </transmission>
         <!-- Link 3/Tibia -->
         <joint name="FT_joint_${suffix}" type="revolute">
             <parent link="femur_${suffix}"/>
             <child link="tibia_${suffix}"/>
-            <origin xyz="${femur_length} 0.00 0.00" rpy="0.00 ${radians(45 + tibia_angle)}  0.00"/>
-            <axis xyz="0.00 ${mirror * 1.00} 0.00"/>
+            <origin xyz="${femur_length} 0.00 0.00" rpy="0.00 0.00 0.00"/>
+            <axis xyz="0.00 1.00 0.00"/>
             <limit lower="${FT_joint_lower_limit}" upper="${FT_joint_upper_limit}" effort="${max_torque}" velocity="${max_velocity}"/>
-            <dynamics damping="${damping}" friction="${friction}" />
+            <!--<dynamics damping="${damping}" friction="${friction}" />-->
         </joint>
         <link name="tibia_${suffix}">
@@ -125,11 +148,22 @@
                 </geometry>
             </collision>
-            <xacro:cylinder_inertial_with_origin mass="${tibia_mass}" radius="0.02" length="${tibia_length}">
-                <origin xyz="${tibia_length/2} 0.00 0.00" rpy="0.00 ${radians(90)} 0.00"/>
-            </xacro:cylinder_inertial_with_origin>
+            <xacro:default_inertial/>
+            <!--<xacro:cylinder_inertial_with_origin mass="${tibia_mass}" radius="0.02" length="${tibia_length}">-->
+                <!--<origin xyz="${tibia_length/2} 0.00 0.00" rpy="0.00 ${radians(90)} 0.00"/>-->
+            <!--</xacro:cylinder_inertial_with_origin>-->
         </link>
         <gazebo reference="tibia_${suffix}">
             <material>Gazebo/Purple</material>
         </gazebo>
+        <transmission name="FT_trans_${suffix}">
+            <type>transmission_interface/SimpleTransmission</type>
+            <joint name="FT_joint_${suffix}">
+                <hardwareInterface>hardware_interface/EffortJointInterface</hardwareInterface>
+            </joint>
+            <actuator name="FT_motor_${suffix}">
+                <hardwareInterface>hardware_interface/EffortJointInterface</hardwareInterface>
+                <mechanicalReduction>1</mechanicalReduction>
+            </actuator>
+        </transmission>
         <!-- Tip/Foot -->
         <joint name="foot_joint_${suffix}" type="fixed">
@@ -154,5 +188,6 @@
                 </geometry>
             </collision>
-            <xacro:sphere_inertial mass="${foot_mass}" radius="0.01"/>
+            <xacro:default_inertial/>
+            <!--<xacro:sphere_inertial mass="${foot_mass}" radius="0.01"/>-->
         </link>
         <gazebo reference="foot_frame_${suffix}">
@@ -164,35 +199,4 @@
             <!--<fdir1 value="1 0 0"/>-->
         </gazebo>
-        <!-- Transmissions -->
-        <transmission name="TC_trans_${suffix}">
-            <type>transmission_interface/SimpleTransmission</type>
-            <joint name="TC_joint_${suffix}">
-                <hardwareInterface>hardware_interface/PositionJointInterface</hardwareInterface>
-            </joint>
-            <actuator name="TC_motor_${suffix}">
-                <hardwareInterface>hardware_interface/PositionJointInterface</hardwareInterface>
-                <mechanicalReduction>1</mechanicalReduction>
-            </actuator>
-        </transmission>
-        <transmission name="CF_trans_${suffix}">
-            <type>transmission_interface/SimpleTransmission</type>
-            <joint name="CF_joint_${suffix}">
-                <hardwareInterface>hardware_interface/PositionJointInterface</hardwareInterface>
-            </joint>
-            <actuator name="CF_motor_${suffix}">
-                <hardwareInterface>hardware_interface/PositionJointInterface</hardwareInterface>
-                <mechanicalReduction>1</mechanicalReduction>
-            </actuator>
-        </transmission>
-        <transmission name="FT_trans_${suffix}">
-            <type>transmission_interface/SimpleTransmission</type>
-            <joint name="FT_joint_${suffix}">
-                <hardwareInterface>hardware_interface/PositionJointInterface</hardwareInterface>
-            </joint>
-            <actuator name="FT_motor_${suffix}">
-                <hardwareInterface>hardware_interface/PositionJointInterface</hardwareInterface>
-                <mechanicalReduction>1</mechanicalReduction>
-            </actuator>
-        </transmission>
     </xacro:macro>
     <xacro:leg suffix="0" x="${corner_x}" y="${corner_y}" angle="${radians(leg_angle)}" mirror="-1"/>

File: src/mildred_description/urdf/variables.xacro (robot description, xacro)
@@ -23,15 +23,21 @@
     <!--<xacro:property name="foot_mass" value="1.0"/>-->
     <!-- http://emanual.robotis.com/docs/en/dxl/x/xl430-w250/#specifications -->
-    <xacro:property name="max_torque" value="100.4"/> <!-- this is stall torque, graph shows 0.84 -->
-    <xacro:property name="max_velocity" value="${((2*pi)/60)*57}"/> <!-- rpm to rad/s -->
+    <xacro:property name="max_torque" value="1.4"/> <!-- this is stall torque, graph shows 0.84 -->
+    <xacro:property name="max_velocity" value="${((2 * pi) / 60) * 57}"/> <!-- rpm to rad/s -->
     <!--<xacro:property name="max_torque" value="10000"/> &lt;!&ndash; fuck it, just move &ndash;&gt;-->
     <!--<xacro:property name="max_velocity" value="100"/> &lt;!&ndash; fuck it, just move &ndash;&gt;-->
     <!-- Joint Properties -->
-    <xacro:property name="TC_joint_lower_limit" value="-1.2"/> # Swapped per side
-    <xacro:property name="TC_joint_upper_limit" value="1.2"/>
-    <xacro:property name="CF_joint_lower_limit" value="-2.8"/> # Under, Inverted per side
-    <xacro:property name="CF_joint_upper_limit" value="1.8"/>
-    <xacro:property name="FT_joint_lower_limit" value="-1.9"/>
-    <xacro:property name="FT_joint_upper_limit" value="3.7"/>
+    <!--<xacro:property name="TC_joint_lower_limit" value="-1.2"/> # Swapped per side-->
+    <!--<xacro:property name="TC_joint_upper_limit" value="1.2"/>-->
+    <!--<xacro:property name="CF_joint_lower_limit" value="-2.8"/> # Under, Inverted per side-->
+    <!--<xacro:property name="CF_joint_upper_limit" value="1.8"/>-->
+    <!--<xacro:property name="FT_joint_lower_limit" value="-1.9"/>-->
+    <!--<xacro:property name="FT_joint_upper_limit" value="3.7"/>-->
+    <xacro:property name="TC_joint_lower_limit" value="-${3.14}"/>
+    <xacro:property name="TC_joint_upper_limit" value="${3.14}"/>
+    <xacro:property name="CF_joint_lower_limit" value="-${3.14}"/>
+    <xacro:property name="CF_joint_upper_limit" value="${3.14}"/>
+    <xacro:property name="FT_joint_lower_limit" value="-${3.14}"/>
+    <xacro:property name="FT_joint_upper_limit" value="${3.14}"/>
     <!--<xacro:property name="damping" value="0.7"/>-->
     <!--<xacro:property name="friction" value="100.0"/>-->
