Commit message: Started getting results tuning the gazebo sim

File: src/mildred_description/urdf/macros.xacro (robot description, xacro)
@@ -10,5 +10,5 @@
         <inertial>
             <mass value="${mass}"/>
-            <inertia ixx="1.0" ixy="0.0" ixz="0.0" iyy="1.0" iyz="0.0" izz="1.0"/>
+            <inertia ixx="0.001" ixy="0.0" ixz="0.0" iyy="0.001" iyz="0.0" izz="0.001"/>
         </inertial>
     </xacro:macro>
@@ -20,65 +20,11 @@
         <!--</inertial>-->
     <!--</xacro:macro>-->
-    <!--<xacro:macro name="sphere_inertial" params="radius mass">-->
-        <!--<inertial>-->
-            <!--<mass value="${mass}" />-->
-            <!--<origin xyz="0 0 0" />-->
-            <!--<inertia ixx="${0.4 * mass * radius * radius}" ixy="0.0" ixz="0.0"-->
-                     <!--iyy="${0.4 * mass * radius * radius}" iyz="0.0"-->
-                     <!--izz="${0.4 * mass * radius * radius}" />-->
-        <!--</inertial>-->
-    <!--</xacro:macro>-->
-    <!--<xacro:macro name="cylinder_inertial" params="radius length mass">-->
-        <!--<inertial>-->
-            <!--<mass value="${mass}" />-->
-            <!--<origin xyz="0 0 0" />-->
-            <!--<inertia ixx="${0.0833333 * mass * (3 * radius * radius + length * length)}" ixy="0.0" ixz="0.0"-->
-                     <!--iyy="${0.0833333 * mass * (3 * radius * radius + length * length)}" iyz="0.0"-->
-                     <!--izz="${0.5 * mass * radius * radius}" />-->
-        <!--</inertial>-->
-    <!--</xacro:macro>-->
-    <!--<xacro:macro name="box_inertial" params="x y z mass">-->
-        <!--<inertial>-->
-            <!--<mass value="${mass}" />-->
-            <!--<origin xyz="0 0 0" />-->
-            <!--<inertia ixx="${0.0833333 * mass * (y*y + z*z)}" ixy="0.0" ixz="0.0"-->
-                     <!--iyy="${0.0833333 * mass * (x*x + z*z)}" iyz="0.0"-->
-                     <!--izz="${0.0833333 * mass * (x*x + y*y)}" />-->
-        <!--</inertial>-->
-    <!--</xacro:macro>-->
-    <!--<xacro:macro name="sphere_inertial_with_origin" params="radius mass *origin">-->
-        <!--<inertial>-->
-            <!--<mass value="${mass}" />-->
-            <!--<xacro:insert_block name="origin" />-->
-            <!--<inertia ixx="${0.4 * mass * radius * radius}" ixy="0.0" ixz="0.0"-->
-                     <!--iyy="${0.4 * mass * radius * radius}" iyz="0.0"-->
-                     <!--izz="${0.4 * mass * radius * radius}" />-->
-        <!--</inertial>-->
-    <!--</xacro:macro>-->
-    <!--<xacro:macro name="cylinder_inertial_with_origin" params="radius length mass *origin">-->
-        <!--<inertial>-->
-            <!--<mass value="${mass}" />-->
-            <!--<xacro:insert_block name="origin" />-->
-            <!--<inertia ixx="${0.0833333 * mass * (3 * radius * radius + length * length)}" ixy="0.0" ixz="0.0"-->
-                     <!--iyy="${0.0833333 * mass * (3 * radius * radius + length * length)}" iyz="0.0"-->
-                     <!--izz="${0.5 * mass * radius * radius}" />-->
-        <!--</inertial>-->
-    <!--</xacro:macro>-->
-    <!--<xacro:macro name="box_inertial_with_origin" params="x y z mass *origin">-->
-        <!--<inertial>-->
-            <!--<mass value="${mass}" />-->
-            <!--<xacro:insert_block name="origin" />-->
-            <!--<inertia ixx="${0.0833333 * mass * (y*y + z*z)}" ixy="0.0" ixz="0.0"-->
-                     <!--iyy="${0.0833333 * mass * (x*x + z*z)}" iyz="0.0"-->
-                     <!--izz="${0.0833333 * mass * (x*x + y*y)}" />-->
-        <!--</inertial>-->
-    <!--</xacro:macro>-->
     <xacro:macro name="sphere_inertial" params="radius mass">
         <inertial>
             <mass value="${mass}" />
             <origin xyz="0 0 0" />
-            <inertia ixx="1.0" ixy="0.0" ixz="0.0"
-                     iyy="1.0" iyz="0.0"
-                     izz="1.0" />
+            <inertia ixx="${0.4 * mass * radius * radius}" ixy="0.0" ixz="0.0"
+                     iyy="${0.4 * mass * radius * radius}" iyz="0.0"
+                     izz="${0.4 * mass * radius * radius}" />
         </inertial>
     </xacro:macro>
@@ -87,7 +33,7 @@
             <mass value="${mass}" />
             <origin xyz="0 0 0" />
-            <inertia ixx="1.0" ixy="0.0" ixz="0.0"
-                     iyy="1.0" iyz="0.0"
-                     izz="1.0" />
+            <inertia ixx="${0.0833333 * mass * (3 * radius * radius + length * length)}" ixy="0.0" ixz="0.0"
+                     iyy="${0.0833333 * mass * (3 * radius * radius + length * length)}" iyz="0.0"
+                     izz="${0.5 * mass * radius * radius}" />
         </inertial>
     </xacro:macro>
@@ -96,7 +42,7 @@
             <mass value="${mass}" />
             <origin xyz="0 0 0" />
-            <inertia ixx="1.0" ixy="0.0" ixz="0.0"
-                     iyy="1.0" iyz="0.0"
-                     izz="1.0" />
+            <inertia ixx="${0.0833333 * mass * (y*y + z*z)}" ixy="0.0" ixz="0.0"
+                     iyy="${0.0833333 * mass * (x*x + z*z)}" iyz="0.0"
+                     izz="${0.0833333 * mass * (x*x + y*y)}" />
         </inertial>
     </xacro:macro>
@@ -105,7 +51,7 @@
             <mass value="${mass}" />
             <xacro:insert_block name="origin" />
-            <inertia ixx="1.0" ixy="0.0" ixz="0.0"
-                     iyy="1.0" iyz="0.0"
-                     izz="1.0" />
+            <inertia ixx="${0.4 * mass * radius * radius}" ixy="0.0" ixz="0.0"
+                     iyy="${0.4 * mass * radius * radius}" iyz="0.0"
+                     izz="${0.4 * mass * radius * radius}" />
         </inertial>
     </xacro:macro>
@@ -114,7 +60,7 @@
             <mass value="${mass}" />
             <xacro:insert_block name="origin" />
-            <inertia ixx="1.0" ixy="0.0" ixz="0.0"
-                     iyy="1.0" iyz="0.0"
-                     izz="1.0" />
+            <inertia ixx="${0.0833333 * mass * (3 * radius * radius + length * length)}" ixy="0.0" ixz="0.0"
+                     iyy="${0.0833333 * mass * (3 * radius * radius + length * length)}" iyz="0.0"
+                     izz="${0.5 * mass * radius * radius}" />
         </inertial>
     </xacro:macro>
@@ -123,7 +69,7 @@
             <mass value="${mass}" />
             <xacro:insert_block name="origin" />
-            <inertia ixx="1.0" ixy="0.0" ixz="0.0"
-                     iyy="1.0" iyz="0.0"
-                     izz="1.0" />
+            <inertia ixx="${0.0833333 * mass * (y*y + z*z)}" ixy="0.0" ixz="0.0"
+                     iyy="${0.0833333 * mass * (x*x + z*z)}" iyz="0.0"
+                     izz="${0.0833333 * mass * (x*x + y*y)}" />
         </inertial>
     </xacro:macro>

File: src/mildred_description/urdf/mildred.urdf.xacro (robot description, xacro)
@@ -17,5 +17,5 @@
             <origin xyz="0.00 0.00 0.00" rpy="0.00 0.00 0.00"/>
             <geometry>
-                <cylinder radius="${thorax_radius}" length="${thorax_height}"/>
+                <mesh filename="package://mildred_description/stl/body.stl" scale="0.001 0.001 0.001"/>
             </geometry>
             <material name="yellow">
@@ -26,8 +26,9 @@
             <origin xyz="0.00 0.00 0.00" rpy="0.00 0.00 0.00"/>
             <geometry>
-                <cylinder radius="${thorax_radius}" length="${thorax_height}"/>
+                <!--<cylinder radius="${thorax_radius}" length="${thorax_height}"/>-->
+                <mesh filename="package://mildred_description/stl/body.stl" scale="0.001 0.001 0.001"/>
             </geometry>
         </collision>
-        <xacro:default_inertial/>
+        <xacro:default_inertial_mass mass="${thorax_mass}"/>
         <!--<xacro:default_inertial mass="${thorax_mass}"/>-->
     </link>
@@ -37,18 +38,46 @@
     <!-- Leg Macro -->
     <xacro:macro name="leg" params="suffix angle x y mirror">
+        <!-- Leg Anchor -->
+        <joint name="leg_joint_${suffix}" type="fixed">
+            <parent link="thorax"/>
+            <child link="leg_${suffix}"/>
+            <origin xyz="${x} ${y} 0.00" rpy="0.00 0.00 ${angle}"/>
+        </joint>
+        <link name="leg_${suffix}">
+            <visual>
+                <origin xyz="0.00 0.00 0.00" rpy="0.00 0.00 ${radians(-90)}"/>
+                <geometry>
+                    <mesh filename="package://mildred_description/stl/xl430.stl" scale="0.001 0.001 0.001"/>
+                </geometry>
+                <material name="red">
+                    <color rgba="255 0 0 1"/>
+                </material>
+            </visual>
+            <collision>
+                <origin xyz="0.00 0.00 0.00" rpy="0.00 0.00 ${radians(-90)}"/>
+                <geometry>
+                    <mesh filename="package://mildred_description/stl/xl430.stl" scale="0.001 0.001 0.001"/>
+                </geometry>
+            </collision>
+            <xacro:default_inertial/>
+        </link>
+        <gazebo reference="leg_${suffix}">
+            <material>Gazebo/Red</material>
+        </gazebo>
         <!-- Link 1/Coxa -->
-        <joint name="TC_joint_${suffix}" type="revolute">
-            <parent link="thorax"/>
+        <joint name="coxa_joint_${suffix}" type="revolute">
+            <parent link="leg_${suffix}"/>
             <child link="coxa_${suffix}"/>
-            <origin xyz="${x} ${y} 0.00" rpy="0.00 0.00 ${angle}"/>
+            <!--<origin xyz="${x} ${y} 0.00" rpy="0.00 0.00 ${angle}"/>-->
+            <origin xyz="0.00 0.00 0.00" rpy="0.00 0.00 0.00"/>
             <axis xyz="0.00 0.00 1.00"/>
-            <limit lower="${TC_joint_lower_limit}" upper="${TC_joint_upper_limit}" effort="${max_torque}" velocity="${max_velocity}"/>
-            <!--<dynamics damping="${damping}" friction="${friction}" />-->
+            <limit lower="${coxa_joint_lower_limit}" upper="${coxa_joint_upper_limit}" effort="${max_torque}" velocity="${max_velocity}"/>
+            <dynamics damping="${damping}" friction="${friction}" />
         </joint>
         <link name="coxa_${suffix}">
             <visual>
-                <origin xyz="${coxa_length/2} 0.00 0.00" rpy="0.00 ${radians(90)} 0.00"/>
-                <geometry>
-                    <cylinder radius="0.02" length="${coxa_length}"/>
+                <origin xyz="0.00 0.00 0.00" rpy="0.00 0.00 ${radians(-90)}"/>
+                <geometry>
+                    <mesh filename="package://mildred_description/stl/coxa.stl" scale="0.001 0.001 0.001"/>
                 </geometry>
                 <material name="blue">
@@ -57,10 +86,12 @@
             </visual>
             <collision>
-                <origin xyz="${coxa_length/2} 0.00 0.00" rpy="0.00 ${radians(90)} 0.00"/>
-                <geometry>
-                    <cylinder radius="0.02" length="${coxa_length}"/>
-                </geometry>
-            </collision>
-            <xacro:default_inertial/>
+                <!--<origin xyz="${coxa_length/2} 0.00 0.00" rpy="0.00 ${radians(90)} 0.00"/>-->
+                <origin xyz="0.00 0.00 0.00" rpy="0.00 0.00 ${radians(-90)}"/>
+                <geometry>
+                    <!--<cylinder radius="0.02" length="${coxa_length}"/>-->
+                    <mesh filename="package://mildred_description/stl/coxa.stl" scale="0.001 0.001 0.001"/>
+                </geometry>
+            </collision>
+            <xacro:default_inertial_mass mass="${coxa_mass}"/>
             <!--<xacro:cylinder_inertial_with_origin mass="${coxa_mass}" radius="0.02" length="${coxa_length}">-->
                 <!--<origin xyz="${coxa_length/2} 0.00 0.00" rpy="0.00 ${radians(90)} 0.00"/>-->
@@ -70,10 +101,10 @@
             <material>Gazebo/Blue</material>
         </gazebo>
-        <transmission name="TC_trans_${suffix}">
+        <transmission name="coxa_trans_${suffix}">
             <type>transmission_interface/SimpleTransmission</type>
-            <joint name="TC_joint_${suffix}">
+            <joint name="coxa_joint_${suffix}">
                 <hardwareInterface>hardware_interface/EffortJointInterface</hardwareInterface>
             </joint>
-            <actuator name="TC_motor_${suffix}">
+            <actuator name="coxa_motor_${suffix}">
                 <hardwareInterface>hardware_interface/EffortJointInterface</hardwareInterface>
                 <mechanicalReduction>1</mechanicalReduction>
@@ -81,17 +112,17 @@
         </transmission>
         <!-- Link 2/Femur -->
-        <joint name="CF_joint_${suffix}" type="revolute">
+        <joint name="femur_joint_${suffix}" type="revolute">
             <parent link="coxa_${suffix}"/>
             <child link="femur_${suffix}"/>
-            <origin xyz="${coxa_length} 0.00 0.00" rpy="0.00 0.00 0.00"/>
+            <origin xyz="${coxa_length} 0.00 ${coxa_height}" rpy="0.00 0.00 0.00"/>
             <axis xyz="0.00 1.00 0.00"/>
-            <limit lower="${CF_joint_lower_limit}" upper="${CF_joint_upper_limit}" effort="${max_torque}" velocity="${max_velocity}"/>
-            <!--<dynamics damping="${damping}" friction="${friction}" />-->
+            <limit lower="${femur_joint_lower_limit}" upper="${femur_joint_upper_limit}" effort="${max_torque}" velocity="${max_velocity}"/>
+            <dynamics damping="${damping}" friction="${friction}" />
         </joint>
         <link name="femur_${suffix}">
             <visual>
-                <origin xyz="${femur_length/2} 0.00 0.00" rpy="0.00 ${radians(90)} 0.00"/>
-                <geometry>
-                    <cylinder radius="0.02" length="${femur_length}"/>
+                <origin xyz="0.00 0.00 0.00" rpy="0.00 0.00 ${radians(-90)}"/>
+                <geometry>
+                    <mesh filename="package://mildred_description/stl/femur.stl" scale="0.001 0.001 0.001"/>
                 </geometry>
                 <material name="blue">
@@ -100,10 +131,12 @@
             </visual>
             <collision>
-                <origin xyz="${femur_length/2} 0.00 0.00" rpy="0.00 ${radians(90)} 0.00"/>
-                <geometry>
-                    <cylinder radius="0.02" length="${femur_length}"/>
-                </geometry>
-            </collision>
-            <xacro:default_inertial/>
+                <!--<origin xyz="${femur_length/2} 0.00 0.00" rpy="0.00 ${radians(90)} 0.00"/>-->
+                <origin xyz="0.00 0.00 0.00" rpy="0.00 0.00 ${radians(-90)}"/>
+                <geometry>
+                    <!--<cylinder radius="0.02" length="${femur_length}"/>-->
+                    <mesh filename="package://mildred_description/stl/femur.stl" scale="0.001 0.001 0.001"/>
+                </geometry>
+            </collision>
+            <xacro:default_inertial_mass mass="${femur_mass}"/>
             <!--<xacro:cylinder_inertial_with_origin mass="${femur_mass}" radius="0.02" length="${femur_length}">-->
                 <!--<origin xyz="${femur_length/2} 0.00 0.00" rpy="0.00 ${radians(90)} 0.00"/>-->
@@ -113,10 +146,10 @@
             <material>Gazebo/Turquoise</material>
         </gazebo>
-        <transmission name="CF_trans_${suffix}">
+        <transmission name="femur_trans_${suffix}">
             <type>transmission_interface/SimpleTransmission</type>
-            <joint name="CF_joint_${suffix}">
+            <joint name="femur_joint_${suffix}">
                 <hardwareInterface>hardware_interface/EffortJointInterface</hardwareInterface>
             </joint>
-            <actuator name="CF_motor_${suffix}">
+            <actuator name="femur_motor_${suffix}">
                 <hardwareInterface>hardware_interface/EffortJointInterface</hardwareInterface>
                 <mechanicalReduction>1</mechanicalReduction>
@@ -124,17 +157,17 @@
         </transmission>
         <!-- Link 3/Tibia -->
-        <joint name="FT_joint_${suffix}" type="revolute">
+        <joint name="tibia_joint_${suffix}" type="revolute">
             <parent link="femur_${suffix}"/>
             <child link="tibia_${suffix}"/>
             <origin xyz="${femur_length} 0.00 0.00" rpy="0.00 0.00 0.00"/>
             <axis xyz="0.00 1.00 0.00"/>
-            <limit lower="${FT_joint_lower_limit}" upper="${FT_joint_upper_limit}" effort="${max_torque}" velocity="${max_velocity}"/>
-            <!--<dynamics damping="${damping}" friction="${friction}" />-->
+            <limit lower="${tibia_joint_lower_limit}" upper="${tibia_joint_upper_limit}" effort="${max_torque}" velocity="${max_velocity}"/>
+            <dynamics damping="${damping}" friction="${friction}" />
         </joint>
         <link name="tibia_${suffix}">
             <visual>
-                <origin xyz="${tibia_length/2} 0.000 0.00" rpy="0.00 ${radians(90)} 0.00"/>
-                <geometry>
-                    <cylinder radius="0.02" length="${tibia_length}"/>
+                <origin xyz="0.00 0.000 0.00" rpy="${radians(tibia_angle)} 0.00 ${radians(-90)}"/>
+                <geometry>
+                    <mesh filename="package://mildred_description/stl/tibia.stl" scale="0.001 0.001 0.001"/>
                 </geometry>
                 <material name="blue">
@@ -143,10 +176,12 @@
             </visual>
             <collision>
-                <origin xyz="${tibia_length/2} 0.000 0.00" rpy="0.00 ${radians(90)} 0.00"/>
-                <geometry>
-                    <cylinder radius="0.02" length="${tibia_length}"/>
-                </geometry>
-            </collision>
-            <xacro:default_inertial/>
+                <!--<origin xyz="${tibia_length/2} 0.000 0.00" rpy="0.00 ${radians(90)} 0.00"/>-->
+                <origin xyz="0.00 0.000 0.00" rpy="${radians(tibia_angle)} 0.00 ${radians(-90)}"/>
+                <geometry>
+                    <!--<cylinder radius="0.02" length="${tibia_length}"/>-->
+                    <mesh filename="package://mildred_description/stl/tibia.stl" scale="0.001 0.001 0.001"/>
+                </geometry>
+            </collision>
+            <xacro:default_inertial_mass mass="${tibia_mass}"/>
             <!--<xacro:cylinder_inertial_with_origin mass="${tibia_mass}" radius="0.02" length="${tibia_length}">-->
                 <!--<origin xyz="${tibia_length/2} 0.00 0.00" rpy="0.00 ${radians(90)} 0.00"/>-->
@@ -156,10 +191,10 @@
             <material>Gazebo/Purple</material>
         </gazebo>
-        <transmission name="FT_trans_${suffix}">
+        <transmission name="tibia_trans_${suffix}">
             <type>transmission_interface/SimpleTransmission</type>
-            <joint name="FT_joint_${suffix}">
+            <joint name="tibia_joint_${suffix}">
                 <hardwareInterface>hardware_interface/EffortJointInterface</hardwareInterface>
             </joint>
-            <actuator name="FT_motor_${suffix}">
+            <actuator name="tibia_motor_${suffix}">
                 <hardwareInterface>hardware_interface/EffortJointInterface</hardwareInterface>
                 <mechanicalReduction>1</mechanicalReduction>
@@ -188,14 +223,14 @@
                 </geometry>
             </collision>
-            <xacro:default_inertial/>
+            <xacro:default_inertial_mass mass="${foot_mass}"/>
             <!--<xacro:sphere_inertial mass="${foot_mass}" radius="0.01"/>-->
         </link>
         <gazebo reference="foot_frame_${suffix}">
             <material>Gazebo/Red</material>
-            <!--<mu1 value="1.0"/>-->
-            <!--<mu2 value="1.0"/>-->
-            <!--<kp value="10000000.0"/>-->
-            <!--<kd value="1.0"/>-->
-            <!--<fdir1 value="1 0 0"/>-->
+            <mu1 value="1.0"/>
+            <mu2 value="1.0"/>
+            <kp value="10000000.0"/>
+            <kd value="1.0"/>
+            <fdir1 value="1 0 0"/>
         </gazebo>
     </xacro:macro>

File: src/mildred_description/urdf/variables.xacro (robot description, xacro)
@@ -7,13 +7,14 @@
     <xacro:property name="thorax_height" value="0.040"/>
     <xacro:property name="thorax_mass" value="0.2"/>
+    <xacro:property name="coxa_height" value="-0.01305"/>
     <xacro:property name="coxa_length" value="0.03525"/>
     <xacro:property name="coxa_mass" value="0.162"/>
     <xacro:property name="femur_length" value="0.0975"/>
-    <xacro:property name="femur_angle" value="39.2"/>
+    <!--<xacro:property name="femur_angle" value="39.2"/>-->
     <xacro:property name="femur_mass" value="0.025981"/>
     <xacro:property name="tibia_length" value="0.195"/>
     <xacro:property name="tibia_angle" value="21.3"/>
     <xacro:property name="tibia_mass" value="0.107208"/>
-    <xacro:property name="foot_radius" value="0.012"/>
+    <xacro:property name="foot_radius" value="0.006"/>
     <xacro:property name="foot_mass" value="0.005"/>
     <!--<xacro:property name="thorax_mass" value="1.0"/>-->
@@ -28,19 +29,19 @@
     <!--<xacro:property name="max_velocity" value="100"/> &lt;!&ndash; fuck it, just move &ndash;&gt;-->
     <!-- Joint Properties -->
-    <!--<xacro:property name="TC_joint_lower_limit" value="-1.2"/> # Swapped per side-->
-    <!--<xacro:property name="TC_joint_upper_limit" value="1.2"/>-->
-    <!--<xacro:property name="CF_joint_lower_limit" value="-2.8"/> # Under, Inverted per side-->
-    <!--<xacro:property name="CF_joint_upper_limit" value="1.8"/>-->
-    <!--<xacro:property name="FT_joint_lower_limit" value="-1.9"/>-->
-    <!--<xacro:property name="FT_joint_upper_limit" value="3.7"/>-->
-    <xacro:property name="TC_joint_lower_limit" value="-${3.14}"/>
-    <xacro:property name="TC_joint_upper_limit" value="${3.14}"/>
-    <xacro:property name="CF_joint_lower_limit" value="-${3.14}"/>
-    <xacro:property name="CF_joint_upper_limit" value="${3.14}"/>
-    <xacro:property name="FT_joint_lower_limit" value="-${3.14}"/>
-    <xacro:property name="FT_joint_upper_limit" value="${3.14}"/>
-    <!--<xacro:property name="damping" value="0.7"/>-->
-    <!--<xacro:property name="friction" value="100.0"/>-->
+    <!--<xacro:property name="coxa_joint_lower_limit" value="-1.2"/> # Swapped per side-->
+    <!--<xacro:property name="coxa_joint_upper_limit" value="1.2"/>-->
+    <!--<xacro:property name="femur_joint_lower_limit" value="-2.8"/> # Under, Inverted per side-->
+    <!--<xacro:property name="femur_joint_upper_limit" value="1.8"/>-->
+    <!--<xacro:property name="tibia_joint_lower_limit" value="-1.9"/>-->
+    <!--<xacro:property name="tibia_joint_upper_limit" value="3.7"/>-->
+    <xacro:property name="coxa_joint_lower_limit" value="-${3.14}"/>
+    <xacro:property name="coxa_joint_upper_limit" value="${3.14}"/>
+    <xacro:property name="femur_joint_lower_limit" value="-${3.14}"/>
+    <xacro:property name="femur_joint_upper_limit" value="${3.14}"/>
+    <xacro:property name="tibia_joint_lower_limit" value="-${3.14}"/>
+    <xacro:property name="tibia_joint_upper_limit" value="${3.14}"/>
     <xacro:property name="damping" value="0"/>
-    <xacro:property name="friction" value="0"/>
+    <xacro:property name="friction" value="1"/>
+    <!--<xacro:property name="damping" value="0"/>-->
+    <!--<xacro:property name="friction" value="0"/>-->
 </robot>
