Commit message: Adding initialization states

File: src/mildred_description/urdf/variables.xacro (robot description, xacro)
@@ -11,5 +11,5 @@
     <xacro:property name="coxa_mass" value="0.162"/>
     <xacro:property name="femur_length" value="0.0975"/>
-    <!--<xacro:property name="femur_angle" value="39.2"/>-->
+    <xacro:property name="femur_angle" value="39.2"/>
     <xacro:property name="femur_mass" value="0.025981"/>
     <xacro:property name="tibia_length" value="0.195"/>

Commit message: Switched from KDL to tf2 vectors

File: src/mildred_description/urdf/variables.xacro (robot description, xacro)
@@ -24,5 +24,5 @@
     <!--<xacro:property name="foot_mass" value="1.0"/>-->
     <!-- http://emanual.robotis.com/docs/en/dxl/x/xl430-w250/#specifications -->
-    <xacro:property name="max_torque" value="1.4"/> <!-- this is stall torque, graph shows 0.84 -->
+    <xacro:property name="max_torque" value="1.4"/> <!-- this is stall torque, graph shows 0.84, stall torque is 1.4 -->
     <xacro:property name="max_velocity" value="${((2 * pi) / 60) * 57}"/> <!-- rpm to rad/s -->
     <!--<xacro:property name="max_torque" value="10000"/> &lt;!&ndash; fuck it, just move &ndash;&gt;-->
