Commit message: Reintroducing old code

File: src/mildred_description/urdf/mildred.urdf.xacro (robot description, xacro)
@@ -5,103 +5,6 @@
        xmlns:interface="http://playerstage.sourceforge.net/gazebo/xmlschema/#interface"
        xmlns:xacro="http://www.ros.org/wiki/xacro">
-    <xacro:property name="thorax_radius" value="0.064"/>
-    <xacro:property name="thorax_height" value="0.040"/>
-    <xacro:property name="coxa_length" value="0.03525"/>
-    <xacro:property name="femur_length" value="0.090"/>
-    <xacro:property name="femur_angle" value="36"/>
-    <xacro:property name="tibia_length" value="0.180"/>
-    <xacro:property name="tibia_angle" value="21"/>
-    <xacro:property name="thorax_mass" value="0.2"/>
-    <xacro:property name="coxa_mass" value="0.162"/>
-    <xacro:property name="femur_mass" value="0.025981"/>
-    <xacro:property name="tibia_mass" value="0.107208"/>
-    <xacro:property name="foot_mass" value="0.01"/>
-    <!--<xacro:property name="thorax_mass" value="2"/>-->
-    <!--<xacro:property name="coxa_mass" value="1.62"/>-->
-    <!--<xacro:property name="femur_mass" value="0.25981"/>-->
-    <!--<xacro:property name="tibia_mass" value="1.07208"/>-->
-    <!--<xacro:property name="foot_mass" value="0.1"/>-->
-    <!--<xacro:property name="thorax_mass" value="1.0"/>-->
-    <!--<xacro:property name="coxa_mass" value="1.0"/>-->
-    <!--<xacro:property name="femur_mass" value="1.0"/>-->
-    <!--<xacro:property name="tibia_mass" value="1.0"/>-->
-    <!--<xacro:property name="foot_mass" value="1.0"/>-->
-    <!-- http://emanual.robotis.com/docs/en/dxl/x/xl430-w250/#specifications -->
-    <!--<xacro:property name="max_torque" value="1.4"/> &lt;!&ndash; this is stall torque, graph shows 0.84 &ndash;&gt;-->
-    <!--<xacro:property name="max_velocity" value="${((2*pi)/60)*57}"/> &lt;!&ndash; rpm to rad/s &ndash;&gt;-->
-    <xacro:property name="max_torque" value="1000"/> <!-- this is stall torque, graph shows 0.84 -->
-    <xacro:property name="max_velocity" value="${((2*pi)/60)*57}"/> <!-- rpm to rad/s -->
-    <!-- Joint Properties -->
-    <xacro:property name="TC_joint_lower_limit" value="-1.4"/>
-    <xacro:property name="TC_joint_upper_limit" value="1.4"/>
-    <xacro:property name="CF_joint_lower_limit" value="-1.6"/>
-    <xacro:property name="CF_joint_upper_limit" value="1.8"/>
-    <xacro:property name="FT_joint_lower_limit" value="-1.7"/>
-    <xacro:property name="FT_joint_upper_limit" value="2.0"/>
-    <xacro:property name="damping" value="0.7"/>
-    <xacro:property name="friction" value="100.0"/>
-    <!--<xacro:property name="max_torque" value="100" /> &lt;!&ndash; this is stall torque, graph shows 0.84 &ndash;&gt;-->
-    <!--<xacro:property name="max_velocity" value="100" /> &lt;!&ndash; rpm to rad/s &ndash;&gt;-->
-    <xacro:macro name="default_inertial" params="mass">
-        <inertial>
-            <mass value="${mass}"/>
-            <!--<inertia ixx="1.0" ixy="0.0" ixz="0.0" iyy="1.0" iyz="0.0" izz="1.0" />-->
-            <inertia ixx="0.001" ixy="0.0" ixz="0.0" iyy="0.001" iyz="0.0" izz="0.001"/>
-        </inertial>
-    </xacro:macro>
-    <xacro:macro name="sphere_inertial" params="radius mass">
-        <inertial>
-            <mass value="${mass}" />
-            <origin xyz="0 0 0" />
-            <inertia ixx="${0.4 * mass * radius * radius}" ixy="0.0" ixz="0.0"
-                     iyy="${0.4 * mass * radius * radius}" iyz="0.0"
-                     izz="${0.4 * mass * radius * radius}" />
-        </inertial>
-    </xacro:macro>
-    <xacro:macro name="cylinder_inertial" params="radius length mass">
-        <inertial>
-            <mass value="${mass}" />
-            <origin xyz="0 0 0" />
-            <inertia ixx="${0.0833333 * mass * (3 * radius * radius + length * length)}" ixy="0.0" ixz="0.0"
-                     iyy="${0.0833333 * mass * (3 * radius * radius + length * length)}" iyz="0.0"
-                     izz="${0.5 * mass * radius * radius}" />
-        </inertial>
-    </xacro:macro>
-    <xacro:macro name="box_inertial" params="x y z mass">
-        <inertial>
-            <mass value="${mass}" />
-            <origin xyz="0 0 0" />
-            <inertia ixx="${0.0833333 * mass * (y*y + z*z)}" ixy="0.0" ixz="0.0"
-                     iyy="${0.0833333 * mass * (x*x + z*z)}" iyz="0.0"
-                     izz="${0.0833333 * mass * (x*x + y*y)}" />
-        </inertial>
-    </xacro:macro>
-    <xacro:macro name="sphere_inertial_with_origin" params="radius mass *origin">
-        <inertial>
-            <mass value="${mass}" />
-            <xacro:insert_block name="origin" />
-            <inertia ixx="${0.4 * mass * radius * radius}" ixy="0.0" ixz="0.0"
-                     iyy="${0.4 * mass * radius * radius}" iyz="0.0"
-                     izz="${0.4 * mass * radius * radius}" />
-        </inertial>
-    </xacro:macro>
-    <xacro:macro name="cylinder_inertial_with_origin" params="radius length mass *origin">
-        <inertial>
-            <mass value="${mass}" />
-            <xacro:insert_block name="origin" />
-            <inertia ixx="${0.0833333 * mass * (3 * radius * radius + length * length)}" ixy="0.0" ixz="0.0"
-                     iyy="${0.0833333 * mass * (3 * radius * radius + length * length)}" iyz="0.0"
-                     izz="${0.5 * mass * radius * radius}" />
-        </inertial>
-    </xacro:macro>
-    <xacro:macro name="box_inertial_with_origin" params="x y z mass *origin">
-        <inertial>
-            <mass value="${mass}" />
-            <xacro:insert_block name="origin" />
-            <inertia ixx="${0.0833333 * mass * (y*y + z*z)}" ixy="0.0" ixz="0.0"
-                     iyy="${0.0833333 * mass * (x*x + z*z)}" iyz="0.0"
-                     izz="${0.0833333 * mass * (x*x + y*y)}" />
-        </inertial>
-    </xacro:macro>
+    <xacro:include filename="$(find mildred_description)/urdf/variables.xacro" />
+    <xacro:include filename="$(find mildred_description)/urdf/macros.xacro" />
     <link name="base_link"/>
     <joint name="thorax_to_base" type="fixed">
@@ -134,35 +37,35 @@
     <xacro:macro name="leg" params="suffix angle x y">
         <!-- Link 0/Body->Leg -->
-        <joint name="leg_joint_${suffix}" type="fixed">
-            <parent link="thorax"/>
-            <child link="leg_${suffix}"/>
-            <origin xyz="0.00 0.00 0.00" rpy="0.00 0.00 ${angle}"/>
-        </joint>
-        <link name="leg_${suffix}">
-            <visual>
-                <origin xyz="${thorax_radius/2} 0.000 0.00" rpy="0.00 ${pi/2} 0.00"/>
-                <geometry>
-                    <cylinder radius="0.005" length="${thorax_radius}"/>
-                </geometry>
-                <material name="blue">
-                    <color rgba="0 0 255 1"/>
-                </material>
-            </visual>
-            <collision>
-                <origin xyz="${thorax_radius/2} 0.000 0.00" rpy="0.00 ${pi/2} 0.00"/>
-                <geometry>
-                    <cylinder radius="0.005" length="${thorax_radius}"/>
-                </geometry>
-            </collision>
-            <xacro:cylinder_inertial mass="0.01" radius="0.005" length="${thorax_radius}"/>
-        </link>
-        <gazebo reference="leg_${suffix}">
-            <material>Gazebo/Blue</material>
-        </gazebo>
+        <!--<joint name="leg_joint_${suffix}" type="fixed">-->
+            <!--<parent link="thorax"/>-->
+            <!--<child link="leg_${suffix}"/>-->
+            <!--<origin xyz="0.00 0.00 0.00" rpy="0.00 0.00 ${angle}"/>-->
+        <!--</joint>-->
+        <!--<link name="leg_${suffix}">-->
+            <!--<visual>-->
+                <!--<origin xyz="${thorax_radius/2} 0.000 0.00" rpy="0.00 ${radians(90)} 0.00"/>-->
+                <!--<geometry>-->
+                    <!--<cylinder radius="0.005" length="${thorax_radius}"/>-->
+                <!--</geometry>-->
+                <!--<material name="blue">-->
+                    <!--<color rgba="0 0 255 1"/>-->
+                <!--</material>-->
+            <!--</visual>-->
+            <!--<collision>-->
+                <!--<origin xyz="${thorax_radius/2} 0.000 0.00" rpy="0.00 ${radians(90)} 0.00"/>-->
+                <!--<geometry>-->
+                    <!--<cylinder radius="0.005" length="${thorax_radius}"/>-->
+                <!--</geometry>-->
+            <!--</collision>-->
+            <!--<xacro:cylinder_inertial mass="0.01" radius="0.005" length="${thorax_radius}"/>-->
+        <!--</link>-->
+        <!--<gazebo reference="leg_${suffix}">-->
+            <!--<material>Gazebo/Blue</material>-->
+        <!--</gazebo>-->
         <!-- Link 1/Coxa -->
         <joint name="TC_joint_${suffix}" type="revolute">
-            <parent link="leg_${suffix}"/>
+            <parent link="thorax"/>
             <child link="coxa_${suffix}"/>
-            <origin xyz="${thorax_radius} 0.00 0.00" rpy="0.00 0.00 0.00"/>
+            <origin xyz="${x} ${y} 0.00" rpy="0.00 0.00 ${angle}"/>
             <axis xyz="0.00 0.00 1.00"/>
             <limit lower="${TC_joint_lower_limit}" upper="${TC_joint_upper_limit}" effort="${max_torque}" velocity="${max_velocity}"/>
@@ -171,7 +74,7 @@
         <link name="coxa_${suffix}">
             <visual>
-                <origin xyz="${coxa_length/2} 0.00 0.00" rpy="0.00 ${pi/2} 0.00"/>
-                <geometry>
-                    <cylinder radius="0.005" length="${coxa_length}"/>
+                <origin xyz="${coxa_length/2} 0.00 0.00" rpy="0.00 ${radians(90)} 0.00"/>
+                <geometry>
+                    <cylinder radius="0.02" length="${coxa_length}"/>
                 </geometry>
                 <material name="blue">
@@ -180,11 +83,11 @@
             </visual>
             <collision>
-                <origin xyz="${coxa_length/2} 0.00 0.00" rpy="0.00 ${pi/2} 0.00"/>
-                <geometry>
-                    <cylinder radius="0.005" length="${coxa_length}"/>
-                </geometry>
-            </collision>
-            <xacro:cylinder_inertial_with_origin mass="${coxa_mass}" radius="0.005" length="${coxa_length}">
-                <origin xyz="${coxa_length/2} 0.00 0.00" rpy="0.00 ${pi/2} 0.00"/>
+                <origin xyz="${coxa_length/2} 0.00 0.00" rpy="0.00 ${radians(90)} 0.00"/>
+                <geometry>
+                    <cylinder radius="0.02" length="${coxa_length}"/>
+                </geometry>
+            </collision>
+            <xacro:cylinder_inertial_with_origin mass="${coxa_mass}" radius="0.02" length="${coxa_length}">
+                <origin xyz="${coxa_length/2} 0.00 0.00" rpy="0.00 ${radians(90)} 0.00"/>
             </xacro:cylinder_inertial_with_origin>
         </link>
@@ -203,7 +106,7 @@
         <link name="femur_${suffix}">
             <visual>
-                <origin xyz="${femur_length/2} 0.00 0.00" rpy="0.00 ${pi/2} 0.00"/>
-                <geometry>
-                    <cylinder radius="0.005" length="${femur_length}"/>
+                <origin xyz="${femur_length/2} 0.00 0.00" rpy="0.00 ${radians(90)} 0.00"/>
+                <geometry>
+                    <cylinder radius="0.02" length="${femur_length}"/>
                 </geometry>
                 <material name="blue">
@@ -212,11 +115,11 @@
             </visual>
             <collision>
-                <origin xyz="${femur_length/2} 0.00 0.00" rpy="0.00 ${pi/2} 0.00"/>
-                <geometry>
-                    <cylinder radius="0.005" length="${femur_length}"/>
-                </geometry>
-            </collision>
-            <xacro:cylinder_inertial_with_origin mass="${femur_mass}" radius="0.005" length="${femur_length}">
-                <origin xyz="${femur_length/2} 0.00 0.00" rpy="0.00 ${pi/2} 0.00"/>
+                <origin xyz="${femur_length/2} 0.00 0.00" rpy="0.00 ${radians(90)} 0.00"/>
+                <geometry>
+                    <cylinder radius="0.02" length="${femur_length}"/>
+                </geometry>
+            </collision>
+            <xacro:cylinder_inertial_with_origin mass="${femur_mass}" radius="0.02" length="${femur_length}">
+                <origin xyz="${femur_length/2} 0.00 0.00" rpy="0.00 ${radians(90)} 0.00"/>
             </xacro:cylinder_inertial_with_origin>
         </link>
@@ -235,7 +138,7 @@
         <link name="tibia_${suffix}">
             <visual>
-                <origin xyz="${tibia_length/2} 0.000 0.00" rpy="0.00 ${pi/2} 0.00"/>
-                <geometry>
-                    <cylinder radius="0.005" length="${tibia_length}"/>
+                <origin xyz="${tibia_length/2} 0.000 0.00" rpy="0.00 ${radians(90)} 0.00"/>
+                <geometry>
+                    <cylinder radius="0.02" length="${tibia_length}"/>
                 </geometry>
                 <material name="blue">
@@ -244,11 +147,11 @@
             </visual>
             <collision>
-                <origin xyz="${tibia_length/2} 0.000 0.00" rpy="0.00 ${pi/2} 0.00"/>
-                <geometry>
-                    <cylinder radius="0.005" length="${tibia_length}"/>
-                </geometry>
-            </collision>
-            <xacro:cylinder_inertial_with_origin mass="${tibia_mass}" radius="0.005" length="${tibia_length}">
-                <origin xyz="${tibia_length/2} 0.00 0.00" rpy="0.00 ${pi/2} 0.00"/>
+                <origin xyz="${tibia_length/2} 0.000 0.00" rpy="0.00 ${radians(90)} 0.00"/>
+                <geometry>
+                    <cylinder radius="0.02" length="${tibia_length}"/>
+                </geometry>
+            </collision>
+            <xacro:cylinder_inertial_with_origin mass="${tibia_mass}" radius="0.02" length="${tibia_length}">
+                <origin xyz="${tibia_length/2} 0.00 0.00" rpy="0.00 ${radians(90)} 0.00"/>
             </xacro:cylinder_inertial_with_origin>
         </link>
@@ -257,29 +160,29 @@
         </gazebo>
         <!-- Tip/Foot -->
-        <!--<joint name="foot_joint_${suffix}" type="fixed">-->
-            <!--<parent link="tibia_${suffix}"/>-->
-            <!--<child link="foot_frame_${suffix}"/>-->
-            <!--<origin xyz="${tibia_length} 0.00 0.00" rpy="0.00 0.00 0.00"/>-->
-        <!--</joint>-->
-        <!--<link name="foot_frame_${suffix}">-->
-            <!--<visual>-->
-                <!--<origin xyz="0 0 0"/>-->
-                <!--<geometry>-->
-                    <!--<sphere radius="0.01"/>-->
-                <!--</geometry>-->
-                <!--<material name="red">-->
-                    <!--<color rgba="255 0 0 1"/>-->
-                <!--</material>-->
-            <!--</visual>-->
-            <!--<collision name="foot_collision">-->
-                <!--<origin xyz="0 0 0"/>-->
-                <!--<geometry>-->
-                    <!--<sphere radius="0.01"/>-->
-                <!--</geometry>-->
-            <!--</collision>-->
-            <!--<xacro:sphere_inertial mass="${foot_mass}" radius="0.01"/>-->
-        <!--</link>-->
-        <!--<gazebo reference="foot_frame_${suffix}">-->
-            <!--<material>Gazebo/Red</material>-->
+        <joint name="foot_joint_${suffix}" type="fixed">
+            <parent link="tibia_${suffix}"/>
+            <child link="foot_frame_${suffix}"/>
+            <origin xyz="${tibia_length} 0.00 0.00" rpy="0.00 0.00 0.00"/>
+        </joint>
+        <link name="foot_frame_${suffix}">
+            <visual>
+                <origin xyz="0 0 0"/>
+                <geometry>
+                    <sphere radius="${foot_radius}"/>
+                </geometry>
+                <material name="red">
+                    <color rgba="255 0 0 1"/>
+                </material>
+            </visual>
+            <collision name="foot_collision">
+                <origin xyz="0 0 0"/>
+                <geometry>
+                    <sphere radius="${foot_radius}"/>
+                </geometry>
+            </collision>
+            <xacro:sphere_inertial mass="${foot_mass}" radius="0.01"/>
+        </link>
+        <gazebo reference="foot_frame_${suffix}">
+            <material>Gazebo/Red</material>
             <!--<mu1 value="1.0"/>-->
             <!--<mu2 value="1.0"/>-->
@@ -287,5 +190,5 @@
             <!--<kd value="1.0"/>-->
             <!--<fdir1 value="1 0 0"/>-->
-        <!--</gazebo>-->
+        </gazebo>
         <!-- Transmissions -->
         <transmission name="TC_trans_${suffix}">
@@ -295,4 +198,5 @@
             </joint>
             <actuator name="TC_motor_${suffix}">
+                <hardwareInterface>hardware_interface/PositionJointInterface</hardwareInterface>
                 <mechanicalReduction>1</mechanicalReduction>
             </actuator>
@@ -304,4 +208,5 @@
             </joint>
             <actuator name="CF_motor_${suffix}">
+                <hardwareInterface>hardware_interface/PositionJointInterface</hardwareInterface>
                 <mechanicalReduction>1</mechanicalReduction>
             </actuator>
@@ -313,14 +218,15 @@
             </joint>
             <actuator name="FT_motor_${suffix}">
+                <hardwareInterface>hardware_interface/PositionJointInterface</hardwareInterface>
                 <mechanicalReduction>1</mechanicalReduction>
             </actuator>
         </transmission>
     </xacro:macro>
-    <xacro:leg suffix="0" x="0" y="0" angle="${pi/4}"/>
-    <xacro:leg suffix="1" x="0" y="0" angle="${pi/2}"/>
-    <xacro:leg suffix="2" x="0" y="0" angle="${3*pi/4}"/>
-    <xacro:leg suffix="3" x="0" y="0" angle="${7*pi/4}"/>
-    <xacro:leg suffix="4" x="0" y="0" angle="${3*pi/2}"/>
-    <xacro:leg suffix="5" x="0" y="0" angle="${5*pi/4}"/>
+    <xacro:leg suffix="0" x="0.050" y="0.065" angle="${radians(leg_angle)}"/>
+    <xacro:leg suffix="1" x="0.064" y="0.00" angle="${radians(0)}"/>
+    <xacro:leg suffix="2" x="0.050" y="-0.065" angle="${radians(-leg_angle)}"/>
+    <xacro:leg suffix="3" x="-0.050" y="0.065" angle="${radians(180 - leg_angle)}"/>
+    <xacro:leg suffix="4" x="-0.064" y="0.00" angle="${radians(180)}"/>
+    <xacro:leg suffix="5" x="-0.050" y="-0.065" angle="${radians(180 + leg_angle)}"/>
     <gazebo>
         <plugin name="gazebo_ros_control" filename="libgazebo_ros_control.so">

Commit message: Calibrating joints and setting up IK

File: src/mildred_description/urdf/mildred.urdf.xacro (robot description, xacro)
@@ -35,5 +35,5 @@
     </gazebo>
     <!-- Leg Macro -->
-    <xacro:macro name="leg" params="suffix angle x y">
+    <xacro:macro name="leg" params="suffix angle x y mirror">
         <!-- Link 0/Body->Leg -->
         <!--<joint name="leg_joint_${suffix}" type="fixed">-->
@@ -99,6 +99,6 @@
             <parent link="coxa_${suffix}"/>
             <child link="femur_${suffix}"/>
-            <origin xyz="${coxa_length} 0.00 0.00" rpy="0.00 0.00 0.00"/>
-            <axis xyz="0.00 -1.00 0.00"/>
+            <origin xyz="${coxa_length} 0.00 0.00" rpy="0.00 ${-radians(femur_angle)} 0.00"/>
+            <axis xyz="0.00 ${mirror * -1.00} 0.00"/>
             <limit lower="${CF_joint_lower_limit}" upper="${CF_joint_upper_limit}" effort="${max_torque}" velocity="${max_velocity}"/>
             <dynamics damping="${damping}" friction="${friction}" />
@@ -131,6 +131,6 @@
             <parent link="femur_${suffix}"/>
             <child link="tibia_${suffix}"/>
-            <origin xyz="${femur_length} 0.00 0.00" rpy="0.00 0.00 0.00"/>
-            <axis xyz="0.00 1.00 0.00"/>
+            <origin xyz="${femur_length} 0.00 0.00" rpy="0.00 ${radians(45 + tibia_angle)}  0.00"/>
+            <axis xyz="0.00 ${mirror * 1.00} 0.00"/>
             <limit lower="${FT_joint_lower_limit}" upper="${FT_joint_upper_limit}" effort="${max_torque}" velocity="${max_velocity}"/>
             <dynamics damping="${damping}" friction="${friction}" />
@@ -223,10 +223,10 @@
         </transmission>
     </xacro:macro>
-    <xacro:leg suffix="0" x="0.050" y="0.065" angle="${radians(leg_angle)}"/>
-    <xacro:leg suffix="1" x="0.064" y="0.00" angle="${radians(0)}"/>
-    <xacro:leg suffix="2" x="0.050" y="-0.065" angle="${radians(-leg_angle)}"/>
-    <xacro:leg suffix="3" x="-0.050" y="0.065" angle="${radians(180 - leg_angle)}"/>
-    <xacro:leg suffix="4" x="-0.064" y="0.00" angle="${radians(180)}"/>
-    <xacro:leg suffix="5" x="-0.050" y="-0.065" angle="${radians(180 + leg_angle)}"/>
+    <xacro:leg suffix="0" x="${corner_x}" y="${corner_y}" angle="${radians(leg_angle)}" mirror="-1"/>
+    <xacro:leg suffix="1" x="${center_x}" y="0.00" angle="${radians(0)}" mirror="-1"/>
+    <xacro:leg suffix="2" x="${corner_x}" y="-${corner_y}" angle="${radians(-leg_angle)}" mirror="-1"/>
+    <xacro:leg suffix="3" x="-${corner_x}" y="-${corner_y}" angle="${radians(180 + leg_angle)}" mirror="1"/>
+    <xacro:leg suffix="4" x="-${center_x}" y="0.00" angle="${radians(180)}" mirror="1"/>
+    <xacro:leg suffix="5" x="-${corner_x}" y="${corner_y}" angle="${radians(180 - leg_angle)}" mirror="1"/>
     <gazebo>
         <plugin name="gazebo_ros_control" filename="libgazebo_ros_control.so">

File: src/mildred_description/urdf/variables.xacro (robot description, xacro)
@@ -1,11 +1,14 @@
 <robot xmlns:xacro="http://www.ros.org/wiki/xacro">
     <xacro:property name="leg_angle" value="45"/>
+    <xacro:property name="corner_x" value="0.059789"/>
+    <xacro:property name="corner_y" value="0.099919"/>
+    <xacro:property name="center_x" value="0.075378"/>
     <xacro:property name="thorax_radius" value="0.064"/>
     <xacro:property name="thorax_height" value="0.040"/>
     <xacro:property name="coxa_length" value="0.03525"/>
-    <xacro:property name="femur_length" value="0.090"/>
-    <!--<xacro:property name="femur_angle" value="36"/>-->
-    <xacro:property name="tibia_length" value="0.180"/>
-    <!--<xacro:property name="tibia_angle" value="21"/>-->
+    <xacro:property name="femur_length" value="0.0975"/>
+    <xacro:property name="femur_angle" value="39.2"/>
+    <xacro:property name="tibia_length" value="0.195"/>
+    <xacro:property name="tibia_angle" value="21.3"/>
     <xacro:property name="thorax_mass" value="0.2"/>
     <xacro:property name="coxa_mass" value="0.162"/>
@@ -25,10 +28,10 @@
     <!--<xacro:property name="max_velocity" value="100"/> &lt;!&ndash; fuck it, just move &ndash;&gt;-->
     <!-- Joint Properties -->
-    <xacro:property name="TC_joint_lower_limit" value="-1.4"/>
-    <xacro:property name="TC_joint_upper_limit" value="1.4"/>
-    <xacro:property name="CF_joint_lower_limit" value="-1.6"/>
+    <xacro:property name="TC_joint_lower_limit" value="-1.2"/> # Swapped per side
+    <xacro:property name="TC_joint_upper_limit" value="1.2"/>
+    <xacro:property name="CF_joint_lower_limit" value="-2.8"/> # Under, Inverted per side
     <xacro:property name="CF_joint_upper_limit" value="1.8"/>
-    <xacro:property name="FT_joint_lower_limit" value="-1.7"/>
-    <xacro:property name="FT_joint_upper_limit" value="2.0"/>
+    <xacro:property name="FT_joint_lower_limit" value="-1.9"/>
+    <xacro:property name="FT_joint_upper_limit" value="3.7"/>
     <!--<xacro:property name="damping" value="0.7"/>-->
     <!--<xacro:property name="friction" value="100.0"/>-->
