Commit message: Brought back the rotation ignoring ik solver

File: src/mildred_description/urdf/mildred.urdf.xacro (robot description, xacro)
@@ -8,5 +8,5 @@
     <xacro:include filename="$(find mildred_description)/urdf/macros.xacro" />
     <link name="base_link"/>
-    <joint name="thorax_to_base" type="fixed">
+    <joint name="base_to_thorax" type="fixed">
         <parent link="base_link"/>
         <child link="thorax"/>
@@ -36,31 +36,4 @@
     <!-- Leg Macro -->
     <xacro:macro name="leg" params="suffix angle x y mirror">
-        <!-- Link 0/Body->Leg -->
-        <!--<joint name="leg_joint_${suffix}" type="fixed">-->
-            <!--<parent link="thorax"/>-->
-            <!--<child link="leg_${suffix}"/>-->
-            <!--<origin xyz="0.00 0.00 0.00" rpy="0.00 0.00 ${angle}"/>-->
-        <!--</joint>-->
-        <!--<link name="leg_${suffix}">-->
-            <!--<visual>-->
-                <!--<origin xyz="${thorax_radius/2} 0.000 0.00" rpy="0.00 ${radians(90)} 0.00"/>-->
-                <!--<geometry>-->
-                    <!--<cylinder radius="0.005" length="${thorax_radius}"/>-->
-                <!--</geometry>-->
-                <!--<material name="blue">-->
-                    <!--<color rgba="0 0 255 1"/>-->
-                <!--</material>-->
-            <!--</visual>-->
-            <!--<collision>-->
-                <!--<origin xyz="${thorax_radius/2} 0.000 0.00" rpy="0.00 ${radians(90)} 0.00"/>-->
-                <!--<geometry>-->
-                    <!--<cylinder radius="0.005" length="${thorax_radius}"/>-->
-                <!--</geometry>-->
-            <!--</collision>-->
-            <!--<xacro:cylinder_inertial mass="0.01" radius="0.005" length="${thorax_radius}"/>-->
-        <!--</link>-->
-        <!--<gazebo reference="leg_${suffix}">-->
-            <!--<material>Gazebo/Blue</material>-->
-        <!--</gazebo>-->
         <!-- Link 1/Coxa -->
         <joint name="TC_joint_${suffix}" type="revolute">

Commit message: Custom IK

File: src/mildred_description/urdf/mildred.urdf.xacro (robot description, xacro)
@@ -20,5 +20,5 @@
             </geometry>
             <material name="yellow">
-                <color rgba="255 255 0 1"/>
+                <color rgba="1.0 1.0 0.0 1.0"/>
             </material>
         </visual>
@@ -39,5 +39,5 @@
     <xacro:macro name="leg" params="suffix angle x y mirror">
         <!-- Leg Anchor -->
-        <joint name="leg_joint_${suffix}" type="fixed">
+        <joint name="hip_joint_${suffix}" type="fixed">
             <parent link="thorax"/>
             <child link="leg_${suffix}"/>
@@ -51,5 +51,5 @@
                 </geometry>
                 <material name="red">
-                    <color rgba="255 0 0 1"/>
+                    <color rgba="1.0 0.0 0.0 1.0"/>
                 </material>
             </visual>
@@ -69,6 +69,4 @@
             <parent link="leg_${suffix}"/>
             <child link="coxa_${suffix}"/>
-            <!--<origin xyz="${x} ${y} 0.00" rpy="0.00 0.00 ${angle}"/>-->
-            <origin xyz="0.00 0.00 0.00" rpy="0.00 0.00 0.00"/>
             <axis xyz="0.00 0.00 1.00"/>
             <limit lower="${coxa_joint_lower_limit}" upper="${coxa_joint_upper_limit}" effort="${max_torque}" velocity="${max_velocity}"/>
@@ -82,12 +80,10 @@
                 </geometry>
                 <material name="blue">
-                    <color rgba="0 0 255 1"/>
-                </material>
-            </visual>
-            <collision>
-                <!--<origin xyz="${coxa_length/2} 0.00 0.00" rpy="0.00 ${radians(90)} 0.00"/>-->
-                <origin xyz="0.00 0.00 0.00" rpy="0.00 0.00 ${radians(-90)}"/>
-                <geometry>
-                    <!--<cylinder radius="0.02" length="${coxa_length}"/>-->
+                    <color rgba="0.0 0.0 1.0 1.0"/>
+                </material>
+            </visual>
+            <collision>
+                <origin xyz="0.00 0.00 0.00" rpy="0.00 0.00 ${radians(-90)}"/>
+                <geometry>
                     <mesh filename="package://mildred_description/stl/coxa.stl" scale="0.001 0.001 0.001"/>
                 </geometry>
@@ -127,12 +123,10 @@
                 </geometry>
                 <material name="blue">
-                    <color rgba="0 127 127 1"/>
-                </material>
-            </visual>
-            <collision>
-                <!--<origin xyz="${femur_length/2} 0.00 0.00" rpy="0.00 ${radians(90)} 0.00"/>-->
-                <origin xyz="0.00 0.00 0.00" rpy="0.00 0.00 ${radians(-90)}"/>
-                <geometry>
-                    <!--<cylinder radius="0.02" length="${femur_length}"/>-->
+                    <color rgba="0.0 0.5 0.5 1.0"/>
+                </material>
+            </visual>
+            <collision>
+                <origin xyz="0.00 0.00 0.00" rpy="0.00 0.00 ${radians(-90)}"/>
+                <geometry>
                     <mesh filename="package://mildred_description/stl/femur.stl" scale="0.001 0.001 0.001"/>
                 </geometry>
@@ -172,12 +166,10 @@
                 </geometry>
                 <material name="blue">
-                    <color rgba="0 0 255 1"/>
-                </material>
-            </visual>
-            <collision>
-                <!--<origin xyz="${tibia_length/2} 0.000 0.00" rpy="0.00 ${radians(90)} 0.00"/>-->
+                    <color rgba="0.0 0.0 1.0 1.0"/>
+                </material>
+            </visual>
+            <collision>
                 <origin xyz="0.00 0.000 0.00" rpy="${radians(tibia_angle)} 0.00 ${radians(-90)}"/>
                 <geometry>
-                    <!--<cylinder radius="0.02" length="${tibia_length}"/>-->
                     <mesh filename="package://mildred_description/stl/tibia.stl" scale="0.001 0.001 0.001"/>
                 </geometry>
@@ -214,5 +206,5 @@
                 </geometry>
                 <material name="red">
-                    <color rgba="255 0 0 1"/>
+                    <color rgba="1.0 0.0 0.0 1.0"/>
                 </material>
             </visual>

File: src/mildred_description/urdf/variables.xacro (robot description, xacro)
@@ -35,10 +35,10 @@
     <!--<xacro:property name="tibia_joint_lower_limit" value="-1.9"/>-->
     <!--<xacro:property name="tibia_joint_upper_limit" value="3.7"/>-->
-    <xacro:property name="coxa_joint_lower_limit" value="-${3.14}"/>
-    <xacro:property name="coxa_joint_upper_limit" value="${3.14}"/>
-    <xacro:property name="femur_joint_lower_limit" value="-${3.14}"/>
-    <xacro:property name="femur_joint_upper_limit" value="${3.14}"/>
-    <xacro:property name="tibia_joint_lower_limit" value="-${3.14}"/>
-    <xacro:property name="tibia_joint_upper_limit" value="${3.14}"/>
+    <xacro:property name="coxa_joint_lower_limit" value="-${pi}"/>
+    <xacro:property name="coxa_joint_upper_limit" value="${pi}"/>
+    <xacro:property name="femur_joint_lower_limit" value="-${pi}"/>
+    <xacro:property name="femur_joint_upper_limit" value="${pi}"/>
+    <xacro:property name="tibia_joint_lower_limit" value="-${pi}"/>
+    <xacro:property name="tibia_joint_upper_limit" value="${pi}"/>
     <xacro:property name="damping" value="0"/>
     <xacro:property name="friction" value="1"/>
